File: pcb/drone-flight-controller.kicad_sch (KiCad schematic)
At the start: 88 parts, among them J1 SWD, J10 CONN_MANDO, J11 OLED, J12 STM32 SPI, J13 STM32 I2C, J14 STM32 USART, J2 Jumper, J3 USB_B_Micro, J4 CONN_MOT_1, J5 CONN_MOT_2, J6 CONN_MOT_3, J7 CONN_MOT_4, J8 XT-60, J9 LIDAR, SW1 TC-6610_C7528713, SW2 TC-6610_C7528713, SW4 SS12D10G5_C7431054, U1 STM32F103R8T6, U10 LM7805_TO220, U11 AMS1117-3.3, U2 MPU-6050, Y1 8MHz, Y2 32.768KHz

Commit message: pcb: resolve L1 - VDDA gets a real 600R ferrite bead and datasheet caps
The VDDA filter's L1 carried the impossible value 27nF since capture.
It is now a Murata BLM15AG601SN1D 600R@100MHz bead (0402, keeping the
assigned footprint), and C8 drops 100nF -> 10nF so VDDA carries exactly
the 10nF + 1uF of DS5319 Fig. 14 p.36. Provenance recorded in
decisions.md: cap values from the datasheet, the bead from ST
application practice - Fig. 14 itself has no bead. Closes the last
electrical unknown; headless ERC identical.
Parts:
- L1: LCSC (none) -> C76884; Manufacturer (none) -> Murata Electronics; Part (none) -> BLM15AG601SN1D
Changed lines of the file:
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@@
 			)
 		)
-		(property "Datasheet" ""
+		(property "Datasheet" "https://www.lcsc.com/datasheet/lcsc_datasheet_2304140030_Murata-Electronics-BLM15AG601SN1D_C76884.pdf"
 			(at 25.4 157.48 0)
 			(hide yes)
@@
 			)
 		)
-		(property "Description" "Inductor, small symbol"
+		(property "Description" "1 300mA 520mΩ 600Ω@100MHz ±25% 0402 Ferrite Beads ROHS"
 			(at 25.4 157.48 0)
 			(hide yes)
@@
 			)
 		)
+    (property "LCSC" "C76884" (at 25.4 157.48 0)
+      (effects (font (size 1.27 1.27)) (hide yes))
+    )
+    (property "Part" "BLM15AG601SN1D" (at 25.4 157.48 0)
+      (effects (font (size 1.27 1.27)) (hide yes))
+    )
+    (property "Manufacturer" "Murata Electronics" (at 25.4 157.48 0)
+      (effects (font (size 1.27 1.27)) (hide yes))
+    )
 		(pin "2"
 		)

Commit message: pcb: source the entire remaining BOM against the LCSC catalog
Jellybean MPN sweep: ~142 refs across 61 groups - every IC, passive,
LED, diode, crystal, RF inductor, ferrite, and connector now carries
LCSC/Part/Manufacturer/Datasheet fields, resolved offline Basic-first.
Crystals were matched on load capacitance to the repo's original
datasheets, the polarized 10uF pair is the exact original tantalum,
and the nRF matching network gets proper RF multilayer parts. Two
physical deltas: Y2's footprint grows 2012 -> 3215 to fit the Basic
Epson FC-135, and FB1/FB2's invalid "100Uhm" value becomes the
sourced 3A 120R power bead. Sourcing gate: PASS, 0 blocking, 26
Extended lines (~$78 max setup). ERC identical.
Parts:
- C1, C10, C16, C17, C19, C2, C3, C4, C5, C9: LCSC (none) -> C1525; Manufacturer (none) -> Samsung Electro-Mechanics; Part (none) -> CL05B104KO5NNNC
- C11, C12: LCSC (none) -> C1554; Manufacturer (none) -> FH(Guangdong Fenghua Advanced Tech); Part (none) -> 0402CG200J500NT
- C13, C14: LCSC (none) -> C32949; Manufacturer (none) -> Samsung Electro-Mechanics; Part (none) -> CL05C100JB5NNNC
- C15: LCSC (none) -> C1531; Manufacturer (none) -> FH(Guangdong Fenghua Advanced Tech); Part (none) -> 0402B222K500NT
- C18, C8: LCSC (none) -> C15195; Manufacturer (none) -> Samsung Electro-Mechanics; Part (none) -> CL05B103KB5NNNC
- C48: LCSC (none) -> C1857; Manufacturer (none) -> FH(Guangdong Fenghua Advanced Tech); Part (none) -> 1206B224K500NT
- C49: LCSC (none) -> C13585; Manufacturer (none) -> Samsung Electro-Mechanics; Part (none) -> CL31A106KBHNNNE
- C50, C51: LCSC (none) -> C7171; Manufacturer (none) -> AVX; Part (none) -> TAJA106K016RNJ
- C6: LCSC (none) -> C307423; Manufacturer (none) -> Samsung Electro-Mechanics; Part (none) -> CL05A475MQ5NRNC
- C7: LCSC (none) -> C52923; Manufacturer (none) -> Samsung Electro-Mechanics; Part (none) -> CL05A105KA5NQNC
- D1, D2: LCSC (none) -> C64885; Manufacturer (none) -> MDD（Microdiode Electronics）; Part (none) -> B5819W
- D14, D9: LCSC (none) -> C12624; Manufacturer (none) -> Hubei KENTO Elec; Part (none) -> KT-0603G
- D4, D5, D6: LCSC (none) -> C2286; Manufacturer (none) -> Hubei KENTO Elec; Part (none) -> KT-0603R
- D7, D8: LCSC (none) -> C2288; Manufacturer (none) -> Hubei KENTO Elec; Part (none) -> KT-0603B
- FB1, FB2: value 100Uhm @ 100Mhz -> 120R@100MHz; LCSC (none) -> C79382; Manufacturer (none) -> Murata Electronics; Part (none) -> BLM21PG121SN1D
- J1, J11, J13, J14: LCSC (none) -> C2691448; Manufacturer (none) -> XFCN; Part (none) -> PZ254V-11-04P
- J10: LCSC (none) -> C492421; Manufacturer (none) -> XFCN; Part (none) -> PZ254V-12-8P
- J12, J9: LCSC (none) -> C492405; Manufacturer (none) -> XFCN; Part (none) -> PZ254V-11-06P
- J2, J4, J5, J6, J7: LCSC (none) -> C2937625; Manufacturer (none) -> XFCN; Part (none) -> PZ254V-11-03P
- J8: LCSC (none) -> C98733; Manufacturer (none) -> Changzhou Amass Elec; Part (none) -> XT60-M.
- R1, R10, R2, R3: LCSC (none) -> C25744; Manufacturer (none) -> UNI-ROYAL(Uniroyal Elec); Part (none) -> 0402WGF1002TCE
- R11, R12, R13: LCSC (none) -> C23241; Manufacturer (none) -> UNI-ROYAL(Uniroyal Elec); Part (none) -> 0603WAF7500T5E
- R14, R15: LCSC (none) -> C22962; Manufacturer (none) -> UNI-ROYAL(Uniroyal Elec); Part (none) -> 0603WAF2200T5E
- R16: LCSC (none) -> C22775; Manufacturer (none) -> UNI-ROYAL(Uniroyal Elec); Part (none) -> 0603WAF1000T5E
- R17: LCSC (none) -> C25792; Manufacturer (none) -> UNI-ROYAL(Uniroyal Elec); Part (none) -> 0402WGF4702TCE
- R18: LCSC (none) -> C25756; Manufacturer (none) -> UNI-ROYAL(Uniroyal Elec); Part (none) -> 0402WGF1502TCE
- R19, R20, R7, R8, R9: LCSC (none) -> C25900; Manufacturer (none) -> UNI-ROYAL(Uniroyal Elec); Part (none) -> 0402WGF4701TCE
- R39: LCSC (none) -> C25076; Manufacturer (none) -> UNI-ROYAL(Uniroyal Elec); Part (none) -> 0402WGF1000TCE
- R4: LCSC (none) -> C25867; Manufacturer (none) -> UNI-ROYAL(Uniroyal Elec); Part (none) -> 0402WGF1501TCE
- R5, R6: LCSC (none) -> C25092; Manufacturer (none) -> UNI-ROYAL(Uniroyal Elec); Part (none) -> 0402WGF220JTCE
- U1: LCSC (none) -> C46034; Manufacturer (none) -> STMicroelectronics; Part (none) -> STM32F103R8T6
- U10: LCSC (none) -> C5189702; Manufacturer (none) -> JSMSEMI; Part (none) -> L7805CV
- U11: LCSC (none) -> C6186; Manufacturer (none) -> Advanced Monolithic Systems; Part (none) -> AMS1117-3.3
- U2: LCSC (none) -> C24112; Manufacturer (none) -> TDK InvenSense; Part (none) -> MPU-6050
- Y1: LCSC (none) -> C115962; Manufacturer (none) -> Yangxing Tech; Part (none) -> X50328MSB2GI
- Y2: footprint Crystal:Crystal_SMD_2012-2Pin_2.0x1.2mm -> Crystal:Crystal_SMD_3215-2Pin_3.2x1.5mm; LCSC (none) -> C32346; Manufacturer (none) -> Seiko Epson; Part (none) -> Q13FC13500004

Commit message: sch: make the USB shield fix immune to symbol updates
'Update Symbols from Library' restored the global Connector lib's stale
SH shield pin for the second time, floating both USB shells again.
Re-apply SH->6 and make it structural: the corrected USB_B_Micro now
lives in the project's custom-symbols library, sym-lib-table registers
it (previously empty), and J3/J16 resolve project-locally - a future
symbol update pulls the corrected copy by construction. Netlist
verified: both shield pins back on GND.
Parts:
- J3: symbol Connector:USB_B_Micro -> custom-symbols:USB_B_Micro
Connections:
- net GND: now also J3.6 (Shield); no longer J3.SH (Shield)
Changed lines of the file:
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@@
 	)
 	(symbol
-		(lib_id "Connector:USB_B_Micro")
+		(lib_id "custom-symbols:USB_B_Micro")
 		(at 110.49 270.51 180)
 		(unit 1)
@@
 		(pin "1"
 		)
-		(pin "SH"
+		(pin "6"
 		)
 		(pin "4"

Commit message: pcb: SW1-SW3 go SMD - TS-1088 (C720477, Basic) supersedes the 6x6 THT tacts
Smaller-footprint request: ~5.6x3.0 mm single-side land vs a 6x6 body with
four through-holes, freeing bottom copper under all three buttons on the
2-layer board. Basic library kills one Extended feeder line and three
hand-solder THT parts. Pad map CLEAN (2 pads <-> 2 pins, no shorted-pair
topology). Board sync via F8 + replace-footprints to follow.
Parts:
- SW1, SW2: value TC-6610_C7528713 -> TS-1088-AR02016_C720477; footprint Button_Switch_THT:SW_PUSH_6mm_H9.5mm -> easyeda:SW-SMD_L3.9-W3.0-P4.45; LCSC C7528713 -> C720477; Manufacturer FG -> XUNPU; Part TC-6610 -6*6*9-260g -> TS-1088-AR02016
Changed lines of the file:
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@@
 			)
 		)
-		(property "Value" "TC-6610_C7528713"
+		(property "Value" "TS-1088-AR02016_C720477"
 			(at 385.064 162.56 90)
 			(hide yes)
@@
 			)
 		)
-		(property "Footprint" "Button_Switch_THT:SW_PUSH_6mm_H9.5mm"
+		(property "Footprint" "easyeda:SW-SMD_L3.9-W3.0-P4.45"
 			(at 387.35 161.29 0)
 			(hide yes)
@@
 			)
 		)
-		(property "Datasheet" "https://wmsc.lcsc.com/wmsc/upload/file/pdf/v2/lcsc/2401191746_FG-TC-6610--6-6-9-260g_C7528713.pdf"
+		(property "Datasheet" "https://www.lcsc.com/datasheet/lcsc_datasheet_2304140030_XUNPU-TS-1088-AR02016_C720477.pdf"
 			(at 387.35 161.29 0)
 			(hide yes)
@@
 			)
 		)
-		(property "LCSC" "C7528713"
+		(property "LCSC" "C720477"
 			(at 382.27 161.29 0)
 			(hide yes)
@@
 			)
 		)
-		(property "Part" "TC-6610 -6*6*9-260g"
+		(property "Part" "TS-1088-AR02016"
 			(at 382.27 161.29 0)
 			(hide yes)
@@
 			)
 		)
-		(property "Manufacturer" "FG"
+		(property "Manufacturer" "XUNPU"
 			(at 382.27 161.29 0)
 			(hide yes)
@@
 			)
 		)
-		(property "Value" "TC-6610_C7528713"
+		(property "Value" "TS-1088-AR02016_C720477"
 			(at 25.4 199.3899 90)
 			(hide yes)
@@
 			)
 		)
-		(property "Footprint" "Button_Switch_THT:SW_PUSH_6mm_H9.5mm"
+		(property "Footprint" "easyeda:SW-SMD_L3.9-W3.0-P4.45"
 			(at 26.67 198.12 0)
 			(hide yes)
@@
 			)
 		)
-		(property "Datasheet" "https://wmsc.lcsc.com/wmsc/upload/file/pdf/v2/lcsc/2401191746_FG-TC-6610--6-6-9-260g_C7528713.pdf"
+		(property "Datasheet" "https://www.lcsc.com/datasheet/lcsc_datasheet_2304140030_XUNPU-TS-1088-AR02016_C720477.pdf"
 			(at 26.67 198.12 0)
 			(hide yes)
@@
 			)
 		)
-		(property "LCSC" "C7528713"
+		(property "LCSC" "C720477"
 			(at 21.59 198.12 0)
 			(hide yes)
@@
 			)
 		)
-		(property "Part" "TC-6610 -6*6*9-260g"
+		(property "Part" "TS-1088-AR02016"
 			(at 21.59 198.12 0)
 			(hide yes)
@@
 			)
 		)
-		(property "Manufacturer" "FG"
+		(property "Manufacturer" "XUNPU"
 			(at 21.59 198.12 0)
 			(hide yes)

Commit message: pcb: SW4 goes right-angle - SS-12D11-G030 (C17179526) supersedes the vertical G5
Edge-actuated master power once the drone is framed; 3A/10k-cycle vs
2A/3k. Pad 2 = middle = common verified against the datasheet PCB layout,
so the +12V/+12C wiring carries over; pads 4/5 are netless bracket slots.
Board F8 sync to follow.
Parts:
- SW4: value SS12D10G5_C7431054 -> SS-12D11-G030_C17179526; footprint easyeda:SW-TH_SHOU-HAN_SS12D10G4 -> easyeda:SW-TH_5P-P4.70_SS-12D11-G030; LCSC C7431054 -> C17179526; Manufacturer SHOU HAN -> G-Switch; Part SS12D10G5 -> SS-12D11-G030
Changed lines of the file:
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@@
 			)
 		)
-		(property "Value" "SS12D10G5_C7431054"
+		(property "Value" "SS-12D11-G030_C17179526"
 			(at 38.1 44.45 0)
 			(show_name no)
@@
 			)
 		)
-		(property "Footprint" "easyeda:SW-TH_SHOU-HAN_SS12D10G4"
+		(property "Footprint" "easyeda:SW-TH_5P-P4.70_SS-12D11-G030"
 			(at 38.1 50.8 0)
 			(hide yes)
@@
 			)
 		)
-		(property "Datasheet" "https://wmsc.lcsc.com/wmsc/upload/file/pdf/v2/lcsc/2311301507_SHOU-HAN-SS12D10G5_C7431054.pdf"
+		(property "Datasheet" "https://wmsc.lcsc.com/wmsc/upload/file/pdf/v2/lcsc/2309150915_G-Switch-SS-12D11-G030_C17179526.pdf"
 			(at 38.1 50.8 0)
 			(hide yes)
@@
 			)
 		)
-		(property "Description" "-25℃~+70℃ 12.7mm 125V 2A 3,000 Cycles 6.7mm SPDT Through Hole 插件,12.7x6.7mm Slide Switches ROHS"
+		(property "Description" "-40℃~+85℃ 10,000 Cycles 13.4mm 250V 3A 6.6mm 8.4mm Black PC Pin Rectangular Columnar Right Angle SPDT 弯插,13.4x6.6mm Slide Switches ROHS"
 			(at 38.1 50.8 0)
 			(hide yes)
@@
 			)
 		)
-		(property "LCSC" "C7431054"
+		(property "LCSC" "C17179526"
 			(at 38.1 50.8 0)
 			(hide yes)
@@
 			)
 		)
-		(property "Part" "SS12D10G5"
+		(property "Part" "SS-12D11-G030"
 			(at 38.1 50.8 0)
 			(hide yes)
@@
 			)
 		)
-		(property "Manufacturer" "SHOU HAN"
+		(property "Manufacturer" "G-Switch"
 			(at 38.1 50.8 0)
 			(hide yes)

Commit message: pcb: SW4 lands on K3-1204D (C145861) - the G030 was too big, so was everything else that could carry the load
Slim 10x2.5 mm vertical slide, 5A/50k cycles: the only part found that
passes both the size requirement and the electrical gate. The hunt is
documented in parts-log: WJ too big, MK-12C02 only 6V, MSK12CO2 only
50mA, SK12D07 killed by its own datasheet (300mA real vs 500mA in the
LCSC listing). Pad 2 = middle = common, wiring unchanged.
Parts:
- SW4: value SS-12D11-G030_C17179526 -> K3-1204D_C145861; footprint easyeda:SW-TH_5P-P4.70_SS-12D11-G030 -> easyeda:SW-TH_K3-1204D; LCSC C17179526 -> C145861; Manufacturer G-Switch -> Korean Hroparts Elec; Part SS-12D11-G030 -> K3-1204D
Changed lines of the file:
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@@
 			)
 		)
-		(property "Value" "SS-12D11-G030_C17179526"
+		(property "Value" "K3-1204D_C145861"
 			(at 38.1 44.45 0)
 			(show_name no)
@@
 			)
 		)
-		(property "Footprint" "easyeda:SW-TH_5P-P4.70_SS-12D11-G030"
+		(property "Footprint" "easyeda:SW-TH_K3-1204D"
 			(at 38.1 50.8 0)
 			(hide yes)
@@
 			)
 		)
-		(property "Datasheet" "https://wmsc.lcsc.com/wmsc/upload/file/pdf/v2/lcsc/2309150915_G-Switch-SS-12D11-G030_C17179526.pdf"
+		(property "Datasheet" "https://www.lcsc.com/datasheet/lcsc_datasheet_2108131730_Korean-Hroparts-Elec-K3-1204D_C145861.pdf"
 			(at 38.1 50.8 0)
 			(hide yes)
@@
 			)
 		)
-		(property "Description" "-40℃~+85℃ 10,000 Cycles 13.4mm 250V 3A 6.6mm 8.4mm Black PC Pin Rectangular Columnar Right Angle SPDT 弯插,13.4x6.6mm Slide Switches ROHS"
+		(property "Description" "-25℃~+80℃ 10mm 120V 2.5mm 50,000 cycles 5A 6mm PC Pin Red SPDT Through Hole 插件,10x2.5mm Slide Switches ROHS"
 			(at 38.1 50.8 0)
 			(hide yes)
@@
 			)
 		)
-		(property "LCSC" "C17179526"
+		(property "LCSC" "C145861"
 			(at 38.1 50.8 0)
 			(hide yes)
@@
 			)
 		)
-		(property "Part" "SS-12D11-G030"
+		(property "Part" "K3-1204D"
 			(at 38.1 50.8 0)
 			(hide yes)
@@
 			)
 		)
-		(property "Manufacturer" "G-Switch"
+		(property "Manufacturer" "Korean Hroparts Elec"
 			(at 38.1 50.8 0)
 			(hide yes)
